File: TweliteEmergencyStop.kicad_pcb (KiCad board)
At the start: 2 copper layers, 45.7 x 58.9 mm, 48 parts, among them J1 BatteryBox, J10 XA02, J11 XA02, J12 XA02, J13 XA02, J14 XA02, J2 BatteryBox, J3 Emergency, J4 Emergency1, J5 Program, J6 Program, J7 Emergency, J8 Emergency2, J9 XA02, U1 TWE-L-WX, U2 TWE-L-DP-W, U3 PC817, U4 PC817, U5 PC817, U6 PC817, U7 R3111N211A, U8 R3111N211A

Commit message: ひらめいた
Parts:
- removed J2: BatteryBox, battery_box:batterybox
- added REF**: MountingHole_3.2mm_M3_DIN965_Pad, MountingHole:MountingHole_3.2mm_M3_DIN965_Pad, F.Cu at (147.6, 92.7)
- added REF**: MountingHole_3.2mm_M3_DIN965_Pad, MountingHole:MountingHole_3.2mm_M3_DIN965_Pad, F.Cu at (239.6, 92.7)
- added REF**: MountingHole_3.2mm_M3_DIN965_Pad, MountingHole:MountingHole_3.2mm_M3_DIN965_Pad, F.Cu at (239.6, 41.7)
- added REF**: MountingHole_3.2mm_M3_DIN965_Pad, MountingHole:MountingHole_3.2mm_M3_DIN965_Pad, F.Cu at (147.6, 41.7)
- moved U1 150.5 mm to (204.1, 25.6)
- moved C2 122.3 mm to (212.2, 93.5), turned to -90 degrees
- moved U2 91.9 mm to (166.4, 78.7), turned to 180 degrees
- moved J1 33.6 mm to (192.9, 94.4)
- moved C1 7.34 mm to (174.7, 93.5), turned to 90 degrees
Connections:
- C2 pad 1: VCCQ -> VCC
- C4 pad 1: VCCQ -> VCC
- J14 pad 2: VCCQ -> VCC
- R1 pad 2: VCCQ -> VCC
- R10 pad 2: VCCQ -> VCC
- R5 pad 2: VCCQ -> VCC
- R6 pad 2: VCCQ -> VCC
- R7 pad 2: VCCQ -> VCC
- R9 pad 2: VCCQ -> VCC
- TP3 pad 1: VCCQ -> VCC
- U1 pad 22: VCCQ -> VCC
- U1 pad 23: VCCQ -> VCC
- U1 pad 24: VCCQ -> VCC
- U1 pad 25: VCCQ -> VCC
- U1 pad 5: VCCQ -> VCC
- U7 pad 2: VCCQ -> VCC
- U8 pad 2: VCCQ -> VCC
Other:
- board size 45.7 x 58.9 mm -> 100 x 65.9 mm

Commit message: 仮
Parts:
- added F1: 350mA, Fuse:Fuse_0805_2012Metric, B.Cu at (161.9, 88.9)
- added F2: 350mA, Fuse:Fuse_0805_2012Metric, B.Cu at (219.7, 78.5)
- added J2: Conn_01x02_Pin, Connector_PinHeader_2.54mm:PinHeader_1x02_P2.54mm_Vertical, F.Cu at (164.4, 92.8)
- added JP3: sw, Jumper:SolderJumper-2_P1.3mm_Open_RoundedPad1.0x1.5mm, B.Cu at (225.4, 64.3)
- added JP4: sw, Jumper:SolderJumper-2_P1.3mm_Open_RoundedPad1.0x1.5mm, B.Cu at (162.3, 53.9)
- C1, C2, C3, JP1, JP2: moved to B.Cu
- J6: value Program -> Conn_01x02_Pin; footprint Connector_PinHeader_2.54mm:PinHeader_1x05_P2.54mm_Vertical -> Connector_PinHeader_2.54mm:PinHeader_1x02_P2.54mm_Vertical
- Low Voltage: renamed from D6; footprint LED_SMD:LED_0603_1608Metric_Pad1.05x0.95mm_HandSolder -> LED_THT:LED_D5.0mm
- Low Voltage: renamed from D5; footprint LED_SMD:LED_0603_1608Metric_Pad1.05x0.95mm_HandSolder -> LED_THT:LED_D5.0mm
- Power: renamed from D3; footprint LED_SMD:LED_0603_1608Metric_Pad1.05x0.95mm_HandSolder -> LED_THT:LED_D5.0mm
- Power: renamed from D4; footprint LED_SMD:LED_0603_1608Metric_Pad1.05x0.95mm_HandSolder -> LED_THT:LED_D5.0mm
- User: renamed from D2; footprint LED_SMD:LED_0603_1608Metric_Pad1.05x0.95mm_HandSolder -> LED_THT:LED_D5.0mm
- User: renamed from D1; footprint LED_SMD:LED_0603_1608Metric_Pad1.05x0.95mm_HandSolder -> LED_THT:LED_D5.0mm
- moved R1 150.8 mm to (231.0, 54.6), turned to 180 degrees
- moved JP1 145.1 mm to (225.5, 68.3)
- moved U8 143.1 mm to (226.5, 80.4), turned to 180 degrees
- moved R6 138.1 mm to (222.8, 57.3), turned to -90 degrees
- moved OUT2 135.7 mm to (222.7, 41.6)
- moved C4 134.8 mm to (221.8, 76.8), turned to 180 degrees
- moved J5 132.4 mm to (233.2, 73.2), turned to 180 degrees
- moved R10 130.0 mm to (226.8, 82.9), turned to 180 degrees
- moved R5 129.2 mm to (214.2, 57.3), turned to -90 degrees
- moved R7 128.6 mm to (226.9, 87.0), turned to 180 degrees
- moved U6 127.6 mm to (222.8, 54.0), turned to 90 degrees
- moved Power 127.5 mm to (231.8, 84.4), turned to -90 degrees
- moved GND 125.6 mm to (233.3, 58.0)
- moved OUT1 125.4 mm to (214.2, 41.6)
- moved Low Voltage 124.5 mm to (231.8, 77.5), turned to -90 degrees
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- renumbered J8 to Em1, J3 to Em1, J7 to Em2, J4 to Em2, TP4 to GND, TP2 to GND, J12 to O2, J11 to OUT1, J9 to OUT1, J10 to OUT2, TP1 to Vcc, TP3 to Vcc
Connections:
- J1 pad 2: VCC -> /pwr
- J13 pad 2: VCC -> /pwr
- J14 pad 2: VCC -> /pwr
- J6 pad 1: GND -> /pwr
- J6 pad 2: /TX1 -> Net-(J6-Pin_2)
- U1 pad 18: unconnected-(U1-DIO16/DI4-Pad18) -> Net-(JP3-B)
- U2 pad 10: /TX1 -> unconnected-(U2-DIO6/TX-Pad10)
- U2 pad 18: unconnected-(U2-DIO16/DI4-Pad18) -> Net-(JP4-B)
- U2 pad 21: /RST1 -> unconnected-(U2-~{RESET}-Pad21)
- U2 pad 3: /RX1 -> unconnected-(U2-DIO7/RX-Pad3)
- U2 pad 7: /PRG1 -> unconnected-(U2-DO1/PWM3-Pad7)
Routing:
- net VCC: track 0.00 -> 119.8 mm, vias 0 -> 4
- net /pwr: track 0.00 -> 63.2 mm
- net /DI2_2: track 0.00 -> 33.4 mm, vias 0 -> 1
- net /DI1_2: track 0.00 -> 31.7 mm, vias 0 -> 2
- net Net-(D2-K): track 0.00 -> 28.8 mm
- net /DO1_2: track 0.00 -> 26.2 mm, vias 0 -> 1
- net /DO2_2: track 0.00 -> 22.5 mm, vias 0 -> 1
- net Net-(D1-K): track 0.00 -> 22.3 mm, vias 0 -> 1
- net /PRG2: track 0.00 -> 17.2 mm, vias 0 -> 1
- net /DI1_1: track 0.00 -> 13.1 mm
- net /RST2: track 0.00 -> 12.9 mm
- net /DO1_1: track 0.00 -> 12.4 mm
- net Net-(J11-Pin_2): track 0.00 -> 11.7 mm
- net Net-(J12-Pin_1): track 0.00 -> 11.4 mm
- net /DI2_1: track 0.00 -> 11.3 mm
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- added copper zone on B.Cu, net GND
- added copper zone on F.Cu, net GND
Other:
- board size 100 x 65.9 mm -> 83.7 x 59 mm
- board text added: "Enable Emergency Led"
- board text added: "GND"
- board text added: "Handset Mode"
- board text added: "PRG"
- board text added: "Power"
- board text added: "RST"
- board text added: "RX"
- board text added: "SW"
- board text added: "TX"
- board text added: "User"
- board text added: "低電圧"
- board text added: "電源"
