File: TweliteEmergencyStop.kicad_sch (KiCad schematic)
At the start: 48 parts, among them J1 BatteryBox, J10 XA02, J11 XA02, J12 XA02, J13 XA02, J14 XA02, J2 BatteryBox, J3 Emergency, J4 Emergency1, J5 Program, J6 Program, J7 Emergency, J8 Emergency2, J9 XA02, U1 TWE-L-WX, U2 TWE-L-DP-W, U3 PC817, U4 PC817, U5 PC817, U6 PC817, U7 R3111N211A, U8 R3111N211A

Commit message: ひらめいた
Parts:
- removed J2: BatteryBox, battery_box:batterybox, symbol Connector_Generic:Conn_01x02
Connections:
- net VCCQ is gone; now on net VCC: C2.1, C4.1, J14.2 (Pin_2), R1.2, R10.2, R5.2, R6.2, R7.2, R9.2, TP3.1, U1.22 (ADC2/AI3), U1.23 (ADC1/AI1), U1.24 (DIO0/AI2), U1.25 (DIO1/AI4), U1.5 (VCC), U7.2 (VDD), U8.2 (VDD)

Commit message: 仮
Parts:
- removed J6: Program, Connector_PinHeader_2.54mm:PinHeader_1x05_P2.54mm_Vertical, symbol Connector:Conn_01x05_Socket
- added F1, F2: 350mA, Fuse:Fuse_0805_2012Metric, symbol Device:Fuse_Small
- added J2, J6: Conn_01x02_Pin, Connector_PinHeader_2.54mm:PinHeader_1x02_P2.54mm_Vertical, symbol Connector:Conn_01x02_Pin
- added JP3, JP4: sw, Jumper:SolderJumper-2_P1.3mm_Open_RoundedPad1.0x1.5mm, symbol Jumper:Jumper_2_Small_Open
- D1, D2, D3, D4, D5, D6: footprint LED_SMD:LED_0603_1608Metric_Pad1.05x0.95mm_HandSolder -> LED_THT:LED_D5.0mm
Connections:
- net DI1_1: now also JP4.1 (A)
- net DI1_2: now also JP3.1 (A)
- net VCC: now also F1.1, F2.1; no longer J1.2 (Pin_2), J13.2 (Pin_2), J14.2 (Pin_2)
- net at U1.18 (DIO16/DI4): now also JP3.2 (B)
- net at U2.18 (DIO16/DI4): now also JP4.2 (B)
- net PRG1: no longer names the net of U2.7 (DO1/PWM3)
- net RST1: no longer names the net of U2.21 (~{RESET})
- net RX1: no longer names the net of U2.3 (DIO7/RX)
- net TX1: no longer names the net of U2.10 (DIO6/TX)
- new net: F2.2, J6.2 (Pin_2)
- new net: F1.2, J2.2 (Pin_2)
- new net pwr: J1.2 (Pin_2), J13.2 (Pin_2), J14.2 (Pin_2), J2.1 (Pin_1), J6.1 (Pin_1)
- no-connect marks 26 -> 28
Other:
- moved on the sheet: D5, D6, J1, J13, J14, J3, J7, R10, R9, U7, U8
